File: isoSPI-M3Y-BMS-PCB.kicad_pcb (KiCad board)
At the start: 4 copper layers, 260 x 113 mm, 383 parts, among them J1 Screw_Terminal_01x04, J10 Screw_Terminal_01x04, J11 Screw_Terminal_01x03, J12 Screw_Terminal_01x08, J13 Conn_02x10_Odd_Even, J14 Screw_Terminal_01x04, J15 USB_C_Receptacle_USB2.0_16P, J16 Conn_01x03, J17 USB_C_Receptacle_USB2.0_16P, J18 USB_C_Receptacle_USB2.0_16P, J2 Conn_02x10_Odd_Even, J3 8P8C_LED_Shielded_x2, J5 OEM Shunt Connector, J6 349128020, J7 OEM HV Sense Connector, J8 OEM Connector, J9 Conn_01x03, Q1 CRSM034N06L2, Q2 CRSM034N06L2, Q3 CRSM034N06L2, Q5 CRSM034N06L2, SW1 TS-1187A-B-A-B, SW2 TS-1187A-B-A-B, SW3 TS-1187A-B-A-B, SW4 TS-1187A-B-A-B, U1 SN74LV1T08DBVR, U10 LTV-217-B-G, U11 RP2354B, U12 ADS1115, U13 ISO1050DUB, U15 SN74LV1T08DBVR, U16 BatMan, U17 TPS5430DDAR, U2 ISO1540, U20 LTV-217-B-G, U21 AMS1117-3.3, U22 F0505S-1WR3, U23 SN74LV1T08DBVR, U24 F0505S-1WR3, U25 SN74LV1T08DBVR, U26 SN74LV1T08DBVR, U27 RP2354B, U28 AM26LV32EIDR, U29 B0505S-3WR2, U3 INA228, U30 ISO1540, U32 SP3485EN-L/TR, U4 ISO1540, U6 F0505S-1WR3, U8 LTV-217-B-G, U9 LTV-217-B-G, Y1 ABM8-272-T3, Y2 ABM8-272-T3

Commit message: connecting main mcu pins
Parts:
- added C73: 100n, Capacitor_SMD:C_0402_1005Metric, F.Cu at (440.3, 246.5)
- added JP13: SolderJumper_3_Open, Jumper:SolderJumper-3_P1.3mm_Open_RoundedPad1.0x1.5mm_NumberLabels, F.Cu at (475.0, 286.3)
- added JP14: SolderJumper_3_Open, Jumper:SolderJumper-3_P1.3mm_Open_RoundedPad1.0x1.5mm_NumberLabels, F.Cu at (475.0, 294.0)
- added R34: 1k, Resistor_SMD:R_0402_1005Metric, F.Cu at (410.9, 236.6)
- added R35: 1k, Resistor_SMD:R_0402_1005Metric, F.Cu at (368.7, 246.3)
- added R57: 1k, Resistor_SMD:R_0402_1005Metric, F.Cu at (451.8, 236.3)
- added R59: 1k, Resistor_SMD:R_0402_1005Metric, F.Cu at (377.1, 235.6)
- added R63: 1k, Resistor_SMD:R_0402_1005Metric, F.Cu at (405.2, 246.2)
- added R64: 1k, Resistor_SMD:R_0402_1005Metric, F.Cu at (405.2, 243.6)
- added TH1: B59451C1130B070, BMS_Library:RV_Disc_D15.5mm_W7.5mm_P5.0mm, F.Cu at (523.3, 263.4)
- added TH2: B59451C1130B070, BMS_Library:RV_Disc_D15.5mm_W7.5mm_P5.0mm, F.Cu at (523.3, 272.4)
- added TH3: B59451C1130B070, BMS_Library:RV_Disc_D15.5mm_W7.5mm_P5.0mm, F.Cu at (523.3, 281.5)
- added TH4: B59451C1130B070, BMS_Library:RV_Disc_D15.5mm_W7.5mm_P5.0mm, F.Cu at (523.3, 290.6)
- added TH5: B59451C1130B070, BMS_Library:RV_Disc_D15.5mm_W7.5mm_P5.0mm, F.Cu at (523.3, 299.6)
- added TH6: B59451C1130B070, BMS_Library:RV_Disc_D15.5mm_W7.5mm_P5.0mm, F.Cu at (523.3, 308.6)
- moved TP7 27.8 mm to (335.3, 249.2), turned to 90 degrees
- moved D26 21.2 mm to (330.1, 250.7), turned to 90 degrees
- moved R75 20.9 mm to (330.1, 247.3), turned to -90 degrees
- moved C53 16.5 mm to (321.1, 254.3), turned to 0 degrees
- moved C50 15.6 mm to (325.5, 254.3), turned to 180 degrees
- moved R67 12.2 mm to (434.2, 244.9), turned to 90 degrees
- moved R66 10.6 mm to (434.3, 248.1), turned to 90 degrees
- moved U21 8.78 mm to (322.3, 248.9), turned to 90 degrees
- moved R29 4.66 mm to (286.7, 294.3)
- moved R28 4.66 mm to (286.7, 297.6)
- moved TP9 2.41 mm to (400.9, 243.8)
- moved R53 1.08 mm to (484.9, 230.7), turned to 0 degrees
- moved R55 0.86 mm to (485.8, 225.2)
- moved D30 0.80 mm to (479.7, 232.8)
- moved FB1 0.80 mm to (474.4, 232.8)
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Connections:
- net /GPIO31 renamed IsoSPI RX Debug
- net /GPIO32 renamed Snooper Debug
- J3 pad 13: Net-(C26-Pad1) -> Net-(J3-Pad13)
- J3 pad 14: Net-(J3-Pad14) -> Net-(C26-Pad1)
- J3 pad 3: GND CAN -> /Wht-Grn
- J3 pad 6: GND CAN -> /Grn
- R140 pad 1: /GPIO45_ADC5 -> 5V Sense
- R144 pad 1: RS232 Tx -> HMI Serial TX
- R146 pad 2: /GPIO45_ADC5 -> 5V Sense
- R148 pad 1: /GPIO46_ADC6 -> Vin Logic Sense
- R150 pad 1: /GPIO46_ADC6 -> Vin Logic Sense
- R28 pad 1: /GPIO47_ADC7 -> VContactor Sense
- R29 pad 1: /GPIO47_ADC7 -> VContactor Sense
- R36 pad 2: Net-(J3-Pad14) -> Net-(J3-Pad13)
- R38 pad 2: unconnected-(R38-Pad2) -> Extra Output 2
- R39 pad 2: unconnected-(R39-Pad2) -> Extra Output 1
- R42 pad 2: Net-(J3-Pad14) -> Net-(J3-Pad13)
- R66 pad 2: /GPIO44_ADC4 -> 3.3V Sense
- R67 pad 1: /GPIO44_ADC4 -> 3.3V Sense
- R94 pad 2: RS232 Rx -> HMI Serial RX
- TP1 pad 1: /GPIO7 -> IsoSPI TX En
- TP1 pad 2: /GPIO8 -> IsoSPI TX Data
- TP17 pad 1: /GPIO10 -> IsoSPI RX H
- TP17 pad 2: /GPIO9 -> IsoSPI RX L
- TP5 pad 1: RS232 Tx -> HMI Serial TX
- TP5 pad 2: RS232 Rx -> HMI Serial RX
- U1 pad 1: /GPIO9 -> IsoSPI RX L
- U1 pad 2: /GPIO10 -> IsoSPI RX H
- U1 pad 4: /GPIO14 -> IsoSPI RX AND
- U10 pad 3: Net-(J3-Pad17) -> Net-(J3-Pad16)
- U10 pad 4: Net-(J3-Pad18) -> Net-(J3-Pad17)
- U11 pad 13: /MCU2_GPIO14 -> C_En
- U11 pad 28: RS232 Tx -> /MCU2_GPIO27
- U11 pad 36: RS232 Rx -> /MCU2_GPIO28
- U11 pad 42: MUC2-MCU1 TX-RX -> /MCU2_GPIO33
- U11 pad 43: MUC1-MCU2 TX-RX -> /MCU2_GPIO34
- U11 pad 77: +3.3V -> /MCU2_GPIO0
- U11 pad 78: /MCU2_GPIO1 -> MUC2-MCU1 TX-RX
- U11 pad 79: /MCU2_GPIO2 -> MUC1-MCU2 TX-RX
- U16 pad 58: BatSPI_MISO -> BatSPI_CS
- U20 pad 3: Net-(J3-Pad15) -> Net-(J3-Pad18)
- U20 pad 4: Net-(J3-Pad16) -> Net-(J3-Pad15)
- U27 pad 27: /GPIO26 -> IsoSPI TX En
- U27 pad 28: RS232 Tx -> IsoSPI TX Data
- U27 pad 36: RS232 Rx -> IsoSPI RX H
- U27 pad 37: /GPIO29 -> IsoSPI RX L
- U27 pad 38: /GPIO30 -> IsoSPI RX AND
- U27 pad 42: MUC1-MCU2 TX-RX -> BatSPI_CS
- U27 pad 43: MUC2-MCU1 TX-RX -> BatSPI_SCK
- U27 pad 45: BatSPI_SCK -> BatSPI_MISO
- U27 pad 46: BatSPI_MOSI -> BatSPI_EN
- U27 pad 47: BatSPI_MISO -> HMI Serial TX
- U27 pad 48: BatSPI_EN -> HMI Serial RX
- U27 pad 49: /GPIO40_ADC0 -> 3.3V Sense
- U27 pad 52: /GPIO41_ADC1 -> 5V Sense
- U27 pad 53: /GPIO42_ADC2 -> Vin Logic Sense
- U27 pad 54: /GPIO43_ADC3 -> VContactor Sense
- U27 pad 77: GND -> /GPIO0
- U28 pad 3: /GPIO9 -> IsoSPI RX L
- U28 pad 5: /GPIO10 -> IsoSPI RX H
- U30 pad 2: RS232 Tx -> HMI Serial TX
- U30 pad 3: RS232 Rx -> HMI Serial RX
- U32 pad 3: /GPIO7 -> IsoSPI TX En
- U32 pad 4: /GPIO8 -> IsoSPI TX Data
Routing:
- net /USB_D-: track 1.23 -> 39.0 mm
- net /USB_D+: track 1.23 -> 39.0 mm
- net +5V: track 46.0 -> 31.0 mm
- net IsoSPI RX L: track 0.00 -> 13.9 mm
- net /GPIO9: track 13.9 -> 0.00 mm
- net /USB2_D+: track 109.8 -> 122.4 mm
- net /USB2_D-: track 109.5 -> 121.8 mm
- net IsoSPI RX H: track 0.00 -> 10.8 mm
- net /GPIO10: track 10.8 -> 0.00 mm
- net Net-(U27-USB_DP): track 0.00 -> 4.28 mm
- net IsoSPI TX En: track 0.00 -> 4.11 mm
- net /GPIO7: track 4.11 -> 0.00 mm
- net Net-(U27-USB_DM): track 0.00 -> 3.93 mm
- net GND: track 42.4 -> 39.0 mm, vias 50 -> 53
- net IsoSPI TX Data: track 0.00 -> 3.28 mm
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Other:
- board text added: "1 2 3 4 5 6 7 8"
- board text removed: "1 2 3 GND 4 5 6 GND 7 8"
