File: isoSPI-M3Y-BMS-PCB.kicad_sch (KiCad schematic)
At the start: 414 parts, among them J1 Screw_Terminal_01x04, J10 Screw_Terminal_01x04, J11 Screw_Terminal_01x03, J12 Screw_Terminal_01x08, J13 Conn_02x10_Odd_Even, J14 Screw_Terminal_01x04, J15 USB_C_Receptacle_USB2.0_16P, J16 Conn_01x03, J17 USB_C_Receptacle_USB2.0_16P, J18 USB_C_Receptacle_USB2.0_16P, J2 Conn_02x10_Odd_Even, J3 8P8C_LED_Shielded_x2, J5 OEM Shunt Connector, J6 349128020, J7 OEM HV Sense Connector, J8 OEM Connector, J9 Conn_01x03, K10 FC Positive, K11 FC Negative, K12 Link Negative, K13 Inverter, K14 Link Positive, K15 Link Negative, K16 FC Positive, K17 FC Negative, K18 Inverter, K9 Link Positive, Q1 CRSM034N06L2, Q2 CRSM034N06L2, Q3 CRSM034N06L2, Q5 CRSM034N06L2, SW1 TS-1187A-B-A-B, SW2 TS-1187A-B-A-B, SW3 TS-1187A-B-A-B, SW4 TS-1187A-B-A-B, U1 SN74LV1T08DBVR, U10 LTV-217-B-G, U11 RP2354B, U12 ADS1115, U13 ISO1050DUB, U15 SN74LV1T08DBVR, U16 BatMan, U17 TPS5430DDAR, U2 ISO1540, U20 LTV-217-B-G, U21 AMS1117-3.3, U22 F0505S-1WR3, U23 SN74LV1T08DBVR, U24 F0505S-1WR3, U25 SN74LV1T08DBVR, U26 SN74LV1T08DBVR, U27 RP2354B, U28 AM26LV32EIDR, U29 B0505S-3WR2, U3 INA228, U30 ISO1540, U32 SP3485EN-L/TR, U4 ISO1540, U6 F0505S-1WR3, U8 LTV-217-B-G, U9 LTV-217-B-G, Y1 ABM8-272-T3, Y2 ABM8-272-T3

Commit message: connecting main mcu pins
Parts:
- added C73: 100n, Capacitor_SMD:C_0402_1005Metric, symbol Device:C
- added JP13, JP14: SolderJumper_3_Open, Jumper:SolderJumper-3_P1.3mm_Open_RoundedPad1.0x1.5mm_NumberLabels, symbol Jumper:SolderJumper_3_Open
- added R34, R35, R57, R59, R63, R64: 1k, Resistor_SMD:R_0402_1005Metric, symbol Device:R
- added TP15: TestPoint_2Pole, bms:TestPoint_2Pads_Pitch2.54mm_Drill0.9mm, symbol Connector:TestPoint_2Pole
- J3: JLCPCB Part # (none) -> C3010546
Connections:
- net MCU2_GPIO1 is gone; now on net MUC2-MCU1 TX-RX: U11.78 (GPIO1)
- net MCU2_GPIO14 is gone; now on net C_En: U11.13 (GPIO14)
- net MCU2_GPIO2 is gone; now on net MUC1-MCU2 TX-RX: U11.79 (GPIO2)
- net +3.3V: now also C73.1, R59.1; no longer U11.77 (GPIO0)
- net BatSPI_CS: now also U16.58 (SPI_MISO), U27.42 (GPIO33)
- net BatSPI_EN: now also U27.46 (GPIO37); no longer U27.48 (GPIO39)
- net BatSPI_MISO: now also U27.45 (GPIO36); no longer U27.47 (GPIO38)
- net BatSPI_SCK: now also U27.43 (GPIO34); no longer U27.45 (GPIO36)
- net CAN H: now also JP13.3 (B), JP14.3 (B)
- net CAN L: now also JP13.1 (A), JP14.1 (A)
- net GND: now also C73.2, R57.1; no longer U27.77 (GPIO0)
- net GND CAN: no longer J3.3, J3.6
- net GPIO1: now also R63.2
- net GPIO10: no longer TP17.1, U1.2, U28.5 (2Y)
- net GPIO14: no longer U1.4
- net GPIO2: now also R64.2
- net GPIO44_ADC4: no longer R66.2, R67.1
- net GPIO45_ADC5: no longer R140.1, R146.2
- net GPIO46_ADC6: no longer R148.1, R150.1
- net GPIO47_ADC7: no longer R28.1, R29.1
- net GPIO7: no longer TP1.1, U32.3 (DE)
- net GPIO8: no longer TP1.2, U32.4 (DI)
- net GPIO9: no longer TP17.2, U1.1, U28.3 (1Y)
- net MCU2_GPIO38: now also R34.2
- net MCU2_GPIO39: now also R35.2
- net MUC1-MCU2 TX-RX: now also R63.1; no longer U11.43 (GPIO34), U27.42 (GPIO33)
- net MUC2-MCU1 TX-RX: now also R64.1; no longer U11.42 (GPIO33), U27.43 (GPIO34)
- net at C26.1, J3.23, U9.2: now also J3.14; no longer J3.13
- net at R36.2, R42.2: now also J3.13; no longer J3.14
- net at U20.3: now also J3.18; no longer J3.15
- net at U20.4: now also J3.15; no longer J3.16
- net at U10.3: now also J3.16; no longer J3.17
- net at U10.4: now also J3.17; no longer J3.18
- net Extra Output 2: now reaches R38.2
- net Extra Output 1: now reaches R39.2
- removed net BatSPI_MOSI: U16.58 (SPI_MISO), U27.46 (GPIO37)
- net GPIO26 renamed IsoSPI TX En
- net IsoSPI TX En: now also TP1.1, U32.3 (DE)
- net GPIO29 renamed IsoSPI RX L
- net IsoSPI RX L: now also TP17.2, U1.1, U28.3 (1Y)
- net GPIO30 renamed IsoSPI RX AND
- net IsoSPI RX AND: now also U1.4
- net GPIO31 renamed IsoSPI RX Debug
- net GPIO32 renamed Snooper Debug
- net GPIO40_ADC0 renamed 3.3V Sense
- net 3.3V Sense: now also R66.2, R67.1
- net GPIO41_ADC1 renamed 5V Sense
- net 5V Sense: now also R140.1, R146.2
- net GPIO42_ADC2 renamed Vin Logic Sense
- net Vin Logic Sense: now also R148.1, R150.1
- net GPIO43_ADC3 renamed VContactor Sense
- net VContactor Sense: now also R28.1, R29.1
- net RS232 Rx renamed HMI Serial RX
- net HMI Serial RX: now also U27.48 (GPIO39), R35.1; no longer U11.36 (GPIO28), U27.36 (GPIO28)
- net RS232 Tx renamed HMI Serial TX
- net HMI Serial TX: now also U27.47 (GPIO38), R34.1; no longer U11.28 (GPIO27), U27.28 (GPIO27)
- new net GPIO0: R57.2, U27.77 (GPIO0)
- new net Grn: J3.6, JP14.2 (C)
- new net IsoSPI RX H: TP17.1, U1.2, U27.36 (GPIO28), U28.5 (2Y)
- new net IsoSPI TX Data: TP1.2, U27.28 (GPIO27), U32.4 (DI)
- new net MCU2_GPIO0: R59.2, U11.77 (GPIO0)
- new net MCU2_GPIO27: U11.28 (GPIO27)
- new net MCU2_GPIO28: U11.36 (GPIO28)
- new net MCU2_GPIO33: U11.42 (GPIO33)
- new net MCU2_GPIO34: U11.43 (GPIO34)
- new net Wht-Grn: J3.3, JP13.2 (C)
Other:
- note added: "Blink Blink"
- note added: "Contactor AND gate enable output"
- note added: "Data must be after En"
- note added: "GPIO4 - GPIO13 on NC header"
- note added: "H must be after L"
- note added: "Main MCU"
- note added: "Supervisor MCU"
- note added: "Would be cool if it alternates with main"
- note removed: "MCU 1 BMS"
- note removed: "MCU 2 Supervisor"
- moved on the sheet: C1, C12, C124, C126, C127, C128, C129, C13, C130, C131, C17, C19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

Commit message: fix typo
Other:
- note added: "L must be after H"
- note removed: "H must be after L"
- moved on the sheet: TP15
Changed lines of the file:
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@@
 	(text "Data must be after En"
 		(exclude_from_sim no)
-		(at 435.864 195.072 0)
+		(at 436.372 196.596 0)
 		(effects
 			(font
@@
 		)
 	)
-	(text "H must be after L"
+	(text "L must be after H"
 		(exclude_from_sim no)
-		(at 434.594 200.152 0)
+		(at 434.086 201.676 0)
 		(effects
 			(font
@@
 	(symbol
 		(lib_id "Connector:TestPoint_2Pole")
-		(at 467.36 231.14 90)
+		(at 481.33 215.9 90)
 		(unit 1)
 		(exclude_from_sim no)
@@
 		(dnp no)
 		(property "Reference" "TP15"
-			(at 470.916 231.394 90)
+			(at 484.886 216.154 90)
 			(effects
 				(font
@@
 		)
 		(property "Value" "TestPoint_2Pole"
-			(at 466.852 247.904 90)
+			(at 480.822 232.664 90)
 			(effects
 				(font
@@
 		)
 		(property "Footprint" "bms:TestPoint_2Pads_Pitch2.54mm_Drill0.9mm"
-			(at 467.36 231.14 0)
+			(at 481.33 215.9 0)
 			(effects
 				(font
@@
 		)
 		(property "Datasheet" "~"
-			(at 467.36 231.14 0)
+			(at 481.33 215.9 0)
 			(effects
 				(font
@@
 		)
 		(property "Description" "2-polar test point"
-			(at 467.36 231.14 0)
+			(at 481.33 215.9 0)
 			(effects
 				(font
