File: isoSPI-M3Y-BMS-PCB.kicad_sch (KiCad schematic)
At the start: 468 parts, among them J1 Screw_Terminal_01x04, J10 Screw_Terminal_01x04, J11 3.81P Screw Terminal, J12 3.81P Screw Terminal, J13 Conn_02x10_Odd_Even, J14 Screw_Terminal_01x04, J15 USB_C_Receptacle_USB2.0_16P, J16 Conn_01x03, J17 USB_C_Receptacle_USB2.0_16P, J18 USB_C_Receptacle_USB2.0_16P, J2 Conn_02x10_Odd_Even, J20 Screw_Terminal_01x04, J3 8P8C_LED_Shielded_x2, J5 OEM Shunt Connector, J6 OEM Connector, J7 OEM HV Sense Connector, J8 OEM Connector, J9 Conn_01x03, K10 FC Positive, K11 FC Negative, K12 Link Negative, K13 Inverter, K14 Link Positive, K15 Link Negative, K16 FC Positive, K17 FC Negative, K18 Inverter, K9 Link Positive, Q1 CRSM034N06L2, Q2 CRSM034N06L2, Q3 CRSM034N06L2, Q5 CRSM034N06L2, SW1 TS-1187A-B-A-B, SW2 TS-1187A-B-A-B, SW3 TS-1187A-B-A-B, SW4 TS-1187A-B-A-B, U1 SN74LV1T08DBVR, U10 LTV-217-B-G, U11 RP2354B, U12 ADS1115, U13 ISO1050DUB, U15 SN74LV1T08DBVR, U16 BatMan, U17 TPS5430DDAR, U2 ISO1540, U20 LTV-217-B-G, U21 AMS1117-3.3, U22 F0505S-1WR3, U23 SN74LV1T08DBVR, U24 F0505S-1WR3, U25 SN74LV1T08DBVR, U26 SN74LV1T08DBVR, U27 RP2354B, U28 AM26LV32EIDR, U29 B0505S-3WR2, U3 INA228, U30 ISO1540, U32 SP3485EN-L/TR, U4 ISO1540, U5 LTV-217-B-G, U6 F0505S-1WR3, U7 LTV-217-B-G, U8 LTV-217-B-G, U9 LTV-217-B-G, Y1 ABM8-272-T3, Y2 ABM8-272-T3

Commit message: more tweaks
Parts:
- added C91, C92: 22uF, Capacitor_SMD:C_0805_2012Metric, symbol Device:C_Small
- added C93, C97: 100nF, Capacitor_SMD:C_0603_1608Metric, symbol Device:C_Small
- added C96: 10uF, Capacitor_SMD:C_0805_2012Metric, symbol Device:C_Small
- added D43: Red, LED_SMD:LED_0805_2012Metric, symbol Device:LED
- added D44: Green, LED_SMD:LED_0805_2012Metric, symbol Device:LED
- added D45, D46: SMB6.8CA, Diode_SMD:D_SMB, symbol Device:D_TVS_Small_Filled
- added D47: White, LED_SMD:LED_0805_2012Metric, symbol Device:LED
- added J4: Screw_Terminal_01x04, Connector_Phoenix_MC:PhoenixContact_MC_1,5_4-G-3.81_1x04_P3.81mm_Horizontal, symbol Connector:Screw_Terminal_01x04
- added L9: 6.8uh, Inductor_SMD:L_Changjiang_FXL0630, symbol Device:L_Ferrite
- added R42, R87: 1k, Resistor_SMD:R_0603_1608Metric, symbol Device:R_Small
- added R86, R88, R91: 10k, Resistor_SMD:R_0603_1608Metric, symbol Device:R_Small
- added R89: 510r, Resistor_SMD:R_0603_1608Metric, symbol Device:R_Small
- added TP39, TP40: TestPoint_2Pole, BMS_Library:TestPoint_2Pads_Pitch2.54mm_Pad1.5_Drill1.0mm, symbol Connector:TestPoint_2Pole
- added TP41: TP, BMS_Library:TestPoint_THTPad_D1.5mm_Drill1.0mm, symbol Connector:TestPoint_Small
- added U14: F0505S-1WR3, BMS_Library:H0505S-1WR2, symbol Converter_DCDC1:TEA1-0505HI
- added U18: ISO1540, Package_SO:SOIC-8_3.9x4.9mm_P1.27mm, symbol Isolator:ISO1540
- added U19: UCC27524D, Package_SO:SOIC-8_3.9x4.9mm_P1.27mm, symbol Driver_FET:UCC27524D
- J16, J9: now not fitted
- L6, L7: FT Rotation Offset (none) -> 180
- U10, U20, U22, U24, U29, U5, U6, U7, U8, U9: FT Rotation Offset 90 -> -90
Connections:
- net +3.3V: now also C93.1, R42.1, U18.1 (VCC1); no longer J13.1 (Pin_1), J13.3 (Pin_3), J2.1 (Pin_1), J2.3 (Pin_3)
- net +5V: now also J13.1 (Pin_1), J13.3 (Pin_3), J2.1 (Pin_1), J2.3 (Pin_3), C91.2, L9.2
- net GND: now also C91.1, C92.1, C93.2, D43.1 (K), U14.2 (-Vin), U18.4 (GND1)
- net GND_RS: now also D45.1 (A1), D46.2 (A2)
- new net: C92.2, L9.1, U14.1 (+Vin)
- new net: D44.2 (A), R88.2
- new net: D47.2 (A), R91.2
- new net: D43.2 (A), R86.2
- new net GND_SX: C96.1, C97.1, D44.1 (K), D47.1 (K), J4.4 (Pin_4), R89.2, TP41.1, U14.5 (-Vout), U18.5 (GND2)
- new net SX Serial 5V: C96.2, C97.2, J4.1 (Pin_1), R87.1, R89.1, R91.1, U14.7 (+Vout), U18.8 (VCC2)
- new net SX Serial RX: R42.2, TP39.2, U18.3 (SCL1)
- new net SX Serial RX Iso: D46.1 (A1), J4.3 (Pin_3), R88.1, TP40.1, U18.6 (SCL2)
- new net SX Serial TX: R86.1, TP39.1, U18.2 (SDA1)
- new net SX Serial TX Iso: D45.2 (A2), J4.2 (Pin_2), R87.2, TP40.2, U18.7 (SDA2)
Other:
- note added: "SX 2012-2021 Serial Interface"
- moved on the sheet: C12, C13, C24, C51, C9, D21, D37, D38, D40, D41, D42, J15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

Commit message: REV 0 Ordered!!!
Parts:
- removed U15, U23, U25, U26: SN74LV1T08DBVR, Package_TO_SOT_SMD:SOT-23-5, symbol 74xGxx:74LVC1G08
- added C98, C99: 10uF, Capacitor_SMD:C_0805_2012Metric, symbol Device:C_Small
- added GPIO44, GPIO45, GPIO46, GPIO47: TP, BMS_Library:TestPoint_THTPad_D1.5mm_Drill1.0mm, symbol Connector:TestPoint_Small
- added R113, R117, R93, R95, R96: 5.1k, Resistor_SMD:R_0603_1608Metric, symbol Device:R_Small
- added R118, R92: 1k, Resistor_SMD:R_0603_1608Metric, symbol Device:R_Small
- added TP42: TestPoint_2Pole, BMS_Library:TestPoint_2Pads_Pitch2.54mm_Pad1.5_Drill1.0mm, symbol Connector:TestPoint_2Pole
- added U15: UCC27524DR, Package_SO:SOIC-8_3.9x4.9mm_P1.27mm, symbol Driver_FET:UCC27524D
- C17, C19, C20, C86: JLCPCB Part # v -> C15849
- C81, C82: value 100nF -> 1nF; footprint Capacitor_SMD:C_0603_1608Metric -> Capacitor_SMD:C_1206_3216Metric; Field6 50V X7R -> 2kV X7R; JLCPCB Part # C14663 -> C9196
- J3: FT Rotation Offset (none) -> 180
- J5: JLCPCB Position Offset (none) -> -3.6,0
- R26, R5, R6, R69: value 100R -> 33R; JLCPCB Part # C22775 -> C23140
- R89: JLCPCB Part # (none) -> C23193
- U1: FT Rotation Offset (none) -> 90
- U19: value UCC27524D -> UCC27524DR; Field6 (none) -> 5A 9ns; JLCPCB Part # (none) -> C465729
Connections:
- net C_En is gone; now on net CTR_EN: JP15.1 (A), R58.2
- net FC-Pos is gone; now on net CTR-FC-Pos: U27.16 (GPIO16)
- net GPIO6 is gone; now on net MAX RX: J2.8 (Pin_8), U27.3 (GPIO6)
- net GPIO7 is gone; now on net SX Serial TX: J2.10 (Pin_10), U27.4 (GPIO7)
- net GPIO8 is gone; now on net SX Serial RX: J2.12 (Pin_12), U27.6 (GPIO8)
- net Pos is gone; now on net CTR-LNK-POS: U27.18 (GPIO18)
- net +5V: now also U19.6 (V_{DD}), C98.2, C99.2, U15.6 (V_{DD}); no longer C81.2, C82.2
- net GND: now also U19.3 (GND), C98.1, C99.1, R113.2, R117.2, R93.2, R95.2, R96.2, U15.3 (GND); no longer C81.1, C82.1
- net GND_RS: no longer D45.1 (A1), D46.2 (A2)
- net GND_SX: now also D45.1 (A1), D46.2 (A2)
- net GPIO44_ADC4: now also GPIO44.1
- net GPIO45_ADC5: now also GPIO45.1
- net GPIO46_ADC6: now also GPIO46.1
- net GPIO47_ADC7: now also GPIO47.1
- net MCU2_GPIO6: now also R118.1
- net MCU2_GPIO8: now also R92.1
- net SX Serial RX: now also R92.2
- net at R4.2, R5.1: now also U15.7 (OUTA)
- net at R25.2, R26.1: now also U19.7 (OUTA)
- net MAX RX: now reaches U28.13 (4Y)
- net MAX RX: now also R118.2
- net at U28.14 (4A): now also C81.2
- net at U28.15 (4B): now also C82.2
- net at R17.2, R6.1: now also U19.5 (OUTB)
- net at R62.2, R69.1: now also U15.5 (OUTB)
- net CTR_EN: now reaches U19.1 (ENA)
- net CTR_EN: now also U19.8 (ENB), R93.1, U15.1 (ENA), U15.8 (ENB)
- net CTR-LNK-POS: now reaches U19.2 (INA)
- net CTR-LNK-POS: now also R95.1
- net CTR-FC-Pos: now reaches U19.4 (INB)
- net CTR-FC-Pos: now also R113.1
- net FC-Neg renamed CTR-FC-NEG
- net CTR-FC-NEG: now also R117.1, U15.4 (INB)
- net Neg renamed CTR-LNK-NEG
- net CTR-LNK-NEG: now also R96.1, U15.2 (INA)
- new net: C81.1, TP42.2
- new net: C82.1, TP42.1
Other:
- note added: "Cells to Link Negative Contactor"
- note added: "Cells to Link Positive Contactor"
- note added: "Gate driver has internal 200k pullup, 2x in parallel = 100k pullup must pull down to always start in off state."
- note added: "Gate drivers have weak 120k pulldown. Make sure theyre off by default"
- note added: "all JLC basic components except: MOSFET, TVS, Gate driver"
- note removed: "Cells Negative Contactor"
- note removed: "Cells Positive Contactor"
- note removed: "Contactor AND gate enable output"
- note removed: "all JLC basic components except: MOSFET, TVS"
- moved on the sheet: C1, C10, C11, C112, C117, C118, C12, C120, C123, C124, C126, C127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

Commit message: working on next revision now
Parts:
- removed R142, R143, R190: 10k, Resistor_SMD:R_0603_1608Metric, symbol Device:R_Small
- added C100: 1uF, Capacitor_SMD:C_0603_1608Metric, symbol Device:C_Small
- added FB2: 600R@100MHz, Inductor_SMD:L_0603_1608Metric_Pad1.05x0.95mm_HandSolder, symbol Device:FerriteBead_Small
- added R119: 5.1k, Resistor_SMD:R_0603_1608Metric, symbol Device:R_Small
- added R120, R121: 24k, Resistor_SMD:R_0603_1608Metric, symbol Device:R_Small
- added TP43, TP44, TP45, TP46, TP47, TP48: TP, BMS_Library:TestPoint_THTPad_D1.5mm_Drill1.0mm, symbol Connector:TestPoint_Small
- J1, J10, J20, J4: footprint Connector_Phoenix_MC:PhoenixContact_MC_1,5_4-G-3.81_1x04_P3.81mm_Horizontal -> BMS_Library:PhoenixContact_MC_1,5_4-G-3.81_1x04_P3.81mm_Horizontal_1.4mmPin
- J11: footprint Connector_Phoenix_MC:PhoenixContact_MC_1,5_2-G-3.81_1x02_P3.81mm_Horizontal -> BMS_Library:PhoenixContact_MC_1,5_2-G-3.81_1x02_P3.81mm_Horizontal_1.4mmPin
- J12: footprint Connector_Phoenix_MC:PhoenixContact_MC_1,5_8-G-3.81_1x08_P3.81mm_Horizontal -> BMS_Library:PhoenixContact_MC_1,5_8-G-3.81_1x08_P3.81mm_Horizontal_1.4mmPin
- R48: value 10k -> 5.1k; JLCPCB Part # C25804 -> C23186
- R56, R77, R79, R83, R88, R91: value 10k -> 24k; JLCPCB Part # C25804 -> C23352
- R81: value 10k -> 24k; footprint Resistor_SMD:R_0603_1608Metric_Pad0.98x0.95mm_HandSolder -> Resistor_SMD:R_0603_1608Metric; JLCPCB Part # C25804 -> C23352
Connections:
- net +5V: now also R56.1
- net CAN 5V: now also R120.1, TP47.1; no longer R77.1
- net GND: now also TP44.1, TP45.1
- net GND CAN: now also TP46.1
- net GND_Shunt: now also C100.1
- net GPIO25: now also R119.1; no longer R48.1
- net HMI Serial RX: now also R35.1, U27.48 (GPIO39); no longer R34.1, U27.47 (GPIO38)
- net HMI Serial TX: now also R34.1, U27.47 (GPIO38); no longer R35.1, U27.48 (GPIO39)
- net HV Sense 5V: now also TP43.1
- net I2C SCL Shunt: now also U27.21 (GPIO21); no longer U27.23 (GPIO23)
- net I2C SCL Vsense: now also U27.23 (GPIO23); no longer U27.22 (GPIO22)
- net I2C SDA Vsense: now also U27.22 (GPIO22); no longer U27.21 (GPIO21)
- net Logic_Input: now also R74.1
- net MCU2_GPIO25: now also R48.1; no longer R56.1
- net SX Serial 5V: now also TP48.1
- net Serial API 5V: now also R77.1
- net Serial API RX: now also R121.1
- net Shunt_5V: now also FB2.1; no longer C28.2, C76.2, R111.1, R14.1, R15.1, R68.1, R79.1, U3.6 (VS), U4.8 (VCC2)
- net V_{in}: no longer R74.1
- net at D38.2 (A): now also R121.2
- net at D23.2 (A): now also R56.2
- net at D33.2 (A): now also R119.2; no longer R48.2
- net at R77.2: now also D40.2 (A); no longer D29.2 (A)
- net at D34.2 (A): now also R48.2; no longer R56.2
- new net: C100.2, C28.2, C76.2, FB2.2, R111.1, R14.1, R15.1, R68.1, R79.1, U3.6 (VS), U4.8 (VCC2)
- new net: D29.2 (A), R120.2
Other:
- note added: "I2C pins cannot be re-assigned"
- note added: "TX must be on this pin"
- moved on the sheet: BT1, BT3, BT4, BT5, BT6, BT7, BT8, BT9, D14, D5, F1, F11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

Commit message: WIP - diverting after this to new mounting holes
Parts:
- removed C13: 100nF, Capacitor_SMD:C_0603_1608Metric, symbol Device:C_Small
- removed C24: 10uF, Capacitor_SMD:C_0805_2012Metric, symbol Device:C_Small
- removed D41, D46: SMB6.8CA, Diode_SMD:D_SMB, symbol Device:D_TVS_Small_Filled
- removed R121, R77: 24k, Resistor_SMD:R_0603_1608Metric, symbol Device:R_Small
- removed R141: 510r, Resistor_SMD:R_0603_1608Metric, symbol Device:R_Small
- removed R94, R97: 1k, Resistor_SMD:R_0603_1608Metric, symbol Device:R_Small
- removed U29: B0505S-3WR2, Converter_DCDC:Converter_DCDC_TRACO_TRA3-xxxx_THT, symbol Converter_DCDC:TMU3-0512
- removed U30: ISO1540, Package_SO:SOIC-8_3.9x4.9mm_P1.27mm, symbol Isolator:ISO1540
- added C101: 100nF, Capacitor_SMD:C_0603_1608Metric, symbol Device:C_Small
- added C102, C103: 100pF, Capacitor_SMD:C_0603_1608Metric, symbol Device:C_Small
- added D41: Red, LED_SMD:LED_0805_2012Metric, symbol Device:LED
- added D46: White, LED_SMD:LED_0805_2012Metric, symbol Device:LED
- added FB3: 120Ω@100MHz, Capacitor_SMD:C_0603_1608Metric, symbol Device:FerriteBead_Small
- added FB4, FB6: 600R@100MHz, Inductor_SMD:L_0603_1608Metric_Pad1.05x0.95mm_HandSolder, symbol Device:FerriteBead_Small
- added FL1: SDCW3225S-2-102TF, BMS_Library:FILTER-SMD_4P-L3.2-W2.5-BL, symbol common-mode-filters:SDCW3225S-2-102TF
- added J19: 8P8C_LED_Shielded_x2, Connector_RJ:RJ45_Amphenol_RJHSE538X-02, symbol Connector:8P8C_LED_Shielded_x2
- added JP16: SolderJumper_2_Bridged, BMS_Library:SolderJumper-2_P1.3mm_Bridged_RoundedPad1.0x1.5mm_thin, symbol Jumper:SolderJumper_2_Bridged
- added PS1: MFM-15-5, Converter_ACDC:Converter_ACDC_MeanWell_MFM-15-xx_THT, symbol Converter_ACDC:MFM-15-5
- added R124: 510r, Resistor_SMD:R_0603_1608Metric, symbol Device:R_Small
- added R125: 24k, Resistor_SMD:R_0603_1608Metric, symbol Device:R_Small
- added R128: 120r, Resistor_SMD:R_1206_3216Metric, symbol Device:R_Small
- added TP49, TP50, TP51, TP52: TP, BMS_Library:TestPoint_THTPad_D1.5mm_Drill1.0mm, symbol Connector:TestPoint_Small
- added TP53: TestPoint_2Pole, BMS_Library:TestPoint_2Pads_Pitch2.54mm_Pad1.5_Drill1.0mm, symbol Connector:TestPoint_2Pole
- added U23: F0505S-1WR3, BMS_Library:H0505S-1WR2, symbol Converter_DCDC1:TEA1-0505HI
- added U25: ISO1050DUB, Package_SO:SOP-8_6.62x9.15mm_P2.54mm, symbol Interface_CAN_LIN:ISO1050DUB
- C12: value 100nF -> 22uF; footprint Capacitor_SMD:C_0603_1608Metric -> Capacitor_SMD:C_0805_2012Metric; Field6 50V X7R -> (none); JLCPCB Part # C14663 -> C45783; Voltage (none) -> 25V X5R
- C3: value 4.7uF 50V -> 22uF; footprint Capacitor_SMD:C_1206_3216Metric -> Capacitor_SMD:C_0805_2012Metric; JLCPCB Part # C29823 -> C45783; Voltage (none) -> 25V X5R
- C4: value 4.7uF 50V -> 100nF; footprint Capacitor_SMD:C_1206_3216Metric -> Capacitor_SMD:C_0603_1608Metric; Field6 (none) -> 50V X7R; JLCPCB Part # C29823 -> C14663
- C51: value 22uF -> 10uF; JLCPCB Part # C45783 -> C440198; Voltage 25V X5R -> 50V X5R
- D37: value Red -> Green; JLCPCB Part # C84256 -> C2297
- D40: value White -> Red; JLCPCB Part # C34499 -> C84256
- J8: Field6 (none) -> 2x M3x6 or M3x8 wood or machine screw - both work
- JP1, JP2, JP7, JP8: footprint Jumper:SolderJumper-3_P1.3mm_Bridged12_RoundedPad1.0x1.5mm_NumberLabels -> BMS_Library:SolderJumper-3_P1.3mm_Bridged12_RoundedPad1.0x1.5mm_NumberLabels
- JP9: footprint Jumper:SolderJumper-2_P1.3mm_Bridged_RoundedPad1.0x1.5mm -> BMS_Library:SolderJumper-2_P1.3mm_Bridged_RoundedPad1.0x1.5mm_thin
- R1: value 150r -> 1k; JLCPCB Part # C22808 -> C21190
- R10: value 150r -> 5.1k; JLCPCB Part # C22808 -> C23186
- R178: Field5 (none) -> Shunt
- R2, R8: value 2.2k -> 47r; JLCPCB Part # C4190 -> C23182
- R7: value 510r -> 1k; JLCPCB Part # C23193 -> C21190
- R9: value 510r -> 24k; JLCPCB Part # C23193 -> C23352
Connections:
- net +3.3V: now also C4.1, D2.2 (A), D28.2 (A), D37.2 (A), D38.2 (A), D40.2 (A), D41.2 (A), U25.1 (VCC1)
- net +5V: now also C3.2, FB3.2
- net 1/2 Vsense: now also R47.2; no longer R47.1
- net CAN 5V: now also FB6.2; no longer C16.2, C6.2, U24.7 (+Vout)
- net CAN Rx: now also R83.2; no longer R83.1
- net CAN Tx: now also R84.2; no longer R84.1
- net GND: now also C12.1, C3.1, C4.2, J15.A1 (GND), J15.A12 (GND), J15.B1 (GND), J15.B12 (GND), J15.S1 (SHIELD), TP30.1, TP50.1, U23.2 (-Vin), U25.4 (GND1); no longer C51.1, D2.1 (K), D28.1 (K), D37.1 (K)
- net GND CAN: now also D42.1 (A1), D45.2 (A2), C102.1, C103.2
- net GND_SX: no longer D45.1 (A1)
- net GND_Shunt: no longer C3.1, C4.2, R7.1, R9.2
- net HMI Serial RX: now also R7.2; no longer TP5.2
- net HMI Serial TX: now also R1.2, R10.2; no longer R144.1, TP5.1
- net MAIN-SUP TX/RX: now also R63.1, TP9.1, U27.79 (GPIO2); no longer R64.1, TP9.2, U27.78 (GPIO1)
- net SUP-MAIN TX/RX: now also R64.1, TP9.2, U27.78 (GPIO1); no longer R63.1, TP9.1, U27.79 (GPIO2)
- net SX Serial TX Iso: no longer D45.2 (A2)
- net Serial API RX: now also R144.2, R7.1; no longer D42.1 (A1)
- net Serial API TX: now also R1.1
- net Shunt Sense +: now also C5.2, U3.10 (Vin+); no longer R1.2, R7.2
- net Shunt Sense -: now also C5.1, U3.9 (Vin-); no longer R10.2, R9.1
- net Shunt_5V: now also C100.2, C28.2, C76.2, FB2.2, R111.1, R14.1, R15.1, R79.1, U3.6 (VS), U4.8 (VCC2), TP49.1; no longer C29.2, FB2.1, U22.7 (+Vout)
- net at L4.1: now also C12.2, U23.1 (+Vin); no longer C51.2
- net at C17.1, C19.1, JP8.1 (A): now also R2.2; no longer U32.7 (B)
- net at C43.1, R103.1, TP10.1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: now also R47.1; no longer R47.2
- net at C20.1, C86.1, JP7.1 (A): now also R8.2; no longer U32.6 (A)
- net at U3.3 (~{Alert}): no longer R68.2
- removed net GND_RS: C12.1, D38.1 (K), D40.1 (K), D42.2 (A2), J15.A1 (GND), J15.A12 (GND), J15.B1 (GND), J15.B12 (GND), J15.S1 (SHIELD), TP30.1
- net GPIO4 renamed CAN2 Tx
- net CAN2 Tx: now also R68.2, TP5.2, U25.3 (TXD)
- net GPIO5 renamed CAN2 Rx
- net CAN2 Rx: now also R9.2, TP5.1, U25.2 (RXD)
- net Serial API 5V: no longer names the net of D21.2 (A)
- net Serial API 5V: now also FB3.1; no longer C12.2
- new net: C101.2, C51.2, FB4.1, U23.7 (+Vout)
- new net: D2.1 (K), R83.1
- new net: FB4.2, R124.1, R125.1, TP52.1, U25.8 (VCC2)
- new net: C16.2, C6.2, FB6.1, U24.7 (+Vout)
- new net: FL1.1, U25.7 (CANH)
- new net: FL1.4, U25.6 (CANL)
- new net: D41.1 (K), R68.1
- new net: D38.1 (K), R144.1
- new net: JP16.1 (A), R128.1
- new net: D46.2 (A), R125.2
- new net: C29.2, FB2.1, U22.7 (+Vout)
- new net: D37.1 (K), R9.1
- new net: R8.1, U32.6 (A)
- new net: R2.1, U32.7 (B)
- new net: D40.1 (K), R10.1
- new net: D28.1 (K), R84.1
- new net CAN2 H: C102.2, D42.2 (A2), FL1.2, J19.16, J19.4, R128.2, TP53.2
- new net CAN2 L: C103.1, D45.1 (A1), FL1.3, J19.17, J19.5, JP16.2 (B), TP53.1
- new net GNDCAN2: C101.1, C51.1, D46.1 (K), J19.15, J19.18, J19.3, J19.6, J19.SH, J19.SH, R124.2, TP51.1, U23.5 (-Vout), U25.5 (GND2)
Other:
- note added: "5V 1A max power for external HMI interface MCU/LCD"
- note added: "API TTL RS232 HMI Interface"
- note added: "Aux Input 3-5V limited by resistor dissipation for higher input voltage use external series resistor"
- note added: "Inter-BMS CAN Interface"
- note added: "PTC max current ~10A Under 1S charge time expected"
- note added: "replace pyro with lower value fuse? pyro is always live"
- note added: "use external NC switch for estop"
- note removed: "5V 600mA max external ESP32 interface"
- note removed: "API TTL RS232 Interface"
- note removed: "Option #2"
- note removed: "PTC max current ~10A Under 1S charge time"
- moved on the sheet: BT6, BT7, BT8, BT9, C14, C52, C62, C9, C91, C92, C93, C96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
